File: gpio-expander.sch (KiCad schematic (older format))
At the start: 13 parts, among them J1 Conn_01x06, J2 Conn_02x07_Odd_Even, J3 Conn_02x04_Odd_Even, U1 TCA9555DBT

Commit message: Rev 1.2
Signed-off-by: Aaron Williams <aaron.w2@gmail.com>
Parts:
- removed JP1, JP2, JP3: SolderJumper_2_Open, SolderJumper:SolderJumper-2_P1.3mm_Open_TrianglePad1.0x1.5mm, symbol Jumper:SolderJumper_2_Open
- added SW1: SW_DIP_x06, Buttons_Switches_SMD:SW_DIP_x6_W5.08mm_Slide_Copal_CHS-A, symbol Switch:SW_DIP_x06
- C1: footprint Capacitors_SMD:C_0603_HandSoldering -> Capacitor_SMD:C_0603_1608Metric
- C2, C3, C4: footprint Capacitors_SMD:C_0805_HandSoldering -> Capacitor_SMD:C_0805_2012Metric
- J1: footprint Connector_PinHeader_2.00mm:PinHeader_1x06_P2.00mm_Horizontal -> Pin_Headers:Pin_Header_Angled_1x06_Pitch2.54mm
- RN1, RN2: footprint Resistors_SMD:R_Array_Convex_4x0603 -> Resistor_SMD:R_Array_Convex_4x0603
Connections:
- wire segments 84 -> 90
Changed lines of the file:
@@
 $EndComp
-$Comp
-L Jumper:SolderJumper_2_Open JP1
-U 1 1 5BA217B2
-P 2300 3950
-F 0 "JP1" H 2050 4000 50  0000 C CNN
-F 1 "SolderJumper_2_Open" H 1550 4000 50  0000 C CNN
-F 2 "SolderJumper:SolderJumper-2_P1.3mm_Open_TrianglePad1.0x1.5mm" H 2300 3950 50  0001 C CNN
-F 3 "~" H 2300 3950 50  0001 C CNN
-	1    2300 3950
-	1    0    0    -1
-$EndComp
-$Comp
-L Jumper:SolderJumper_2_Open JP2
-U 1 1 5BA21820
-P 2300 4050
-F 0 "JP2" H 2050 4100 50  0000 C CNN
-F 1 "SolderJumper_2_Open" H 1550 4100 50  0000 C CNN
-F 2 "SolderJumper:SolderJumper-2_P1.3mm_Open_TrianglePad1.0x1.5mm" H 2300 4050 50  0001 C CNN
-F 3 "~" H 2300 4050 50  0001 C CNN
-	1    2300 4050
-	1    0    0    -1
-$EndComp
-$Comp
-L Jumper:SolderJumper_2_Open JP3
-U 1 1 5BA21836
-P 2300 4150
-F 0 "JP3" H 2050 4200 50  0000 C CNN
-F 1 "SolderJumper_2_Open" H 1550 4200 50  0000 C CNN
-F 2 "SolderJumper:SolderJumper-2_P1.3mm_Open_TrianglePad1.0x1.5mm" H 2300 4150 50  0001 C CNN
-F 3 "~" H 2300 4150 50  0001 C CNN
-	1    2300 4150
-	1    0    0    -1
-$EndComp
-Wire Wire Line
-	2150 3950 2150 4050
-Wire Wire Line
-	2150 4050 2150 4150
-Connection ~ 2150 4050
-$Comp
-L power:GND #PWR014
-U 1 1 5BA219EF
-P 2150 4500
-F 0 "#PWR014" H 2150 4250 50  0001 C CNN
-F 1 "GND" H 2155 4327 50  0000 C CNN
-F 2 "" H 2150 4500 50  0001 C CNN
-F 3 "" H 2150 4500 50  0001 C CNN
-	1    2150 4500
-	1    0    0    -1
-$EndComp
-Wire Wire Line
-	2150 4150 2150 4500
-Connection ~ 2150 4150
 $Comp
 L power:GND #PWR013
@@
 F 0 "J1" H 1920 2225 50  0000 C CNN
 F 1 "Conn_01x06" H 1920 2316 50  0000 C CNN
-F 2 "Connector_PinHeader_2.00mm:PinHeader_1x06_P2.00mm_Horizontal" H 2000 2750 50  0001 C CNN
+F 2 "Pin_Headers:Pin_Header_Angled_1x06_Pitch2.54mm" H 2000 2750 50  0001 C CNN
 F 3 "~" H 2000 2750 50  0001 C CNN
 	1    2000 2750
@@
 Wire Wire Line
 	2250 2450 2200 2450
-Wire Wire Line
-	2550 2050 2250 2050
-Connection ~ 2250 2050
 $Comp
 L power:GND #PWR08
@@
 F 0 "C1" H 4592 1296 50  0000 L CNN
 F 1 "1uF" H 4592 1205 50  0000 L CNN
-F 2 "Capacitors_SMD:C_0603_HandSoldering" H 4500 1250 50  0001 C CNN
+F 2 "Capacitor_SMD:C_0603_1608Metric" H 4500 1250 50  0001 C CNN
 F 3 "~" H 4500 1250 50  0001 C CNN
 	1    4500 1250
@@
 F 0 "C2" H 5042 1296 50  0000 L CNN
 F 1 "10uF" H 5042 1205 50  0000 L CNN
-F 2 "Capacitors_SMD:C_0805_HandSoldering" H 4950 1250 50  0001 C CNN
+F 2 "Capacitor_SMD:C_0805_2012Metric" H 4950 1250 50  0001 C CNN
 F 3 "~" H 4950 1250 50  0001 C CNN
 	1    4950 1250
@@
 F 0 "RN1" H 2938 2296 50  0000 L CNN
 F 1 "10k" H 2938 2205 50  0000 L CNN
-F 2 "Resistors_SMD:R_Array_Convex_4x0603" V 3025 2250 50  0001 C CNN
+F 2 "Resistor_SMD:R_Array_Convex_4x0603" V 3025 2250 50  0001 C CNN
 F 3 "~" H 2750 2250 50  0001 C CNN
 	1    2750 2250
@@
 $EndComp
 Wire Wire Line
-	2550 2050 2650 2050
-Connection ~ 2550 2050
-Wire Wire Line
-	2650 2050 2750 2050
-Connection ~ 2650 2050
-Wire Wire Line
-	2750 2050 2850 2050
-Connection ~ 2750 2050
-Wire Wire Line
 	2450 4050 2650 4050
 $Comp
 L Device:R_Pack04 RN2
 U 1 1 5BA42F5D
-P 2750 3650
-F 0 "RN2" H 2938 3696 50  0000 L CNN
-F 1 "10k" H 2950 3600 50  0000 L CNN
-F 2 "Resistors_SMD:R_Array_Convex_4x0603" V 3025 3650 50  0001 C CNN
-F 3 "~" H 2750 3650 50  0001 C CNN
-	1    2750 3650
+P 2650 4500
+F 0 "RN2" H 2838 4546 50  0000 L CNN
+F 1 "10k" H 2850 4450 50  0000 L CNN
+F 2 "Resistor_SMD:R_Array_Convex_4x0603" V 2925 4500 50  0001 C CNN
+F 3 "~" H 2650 4500 50  0001 C CNN
+	1    2650 4500
 	1    0    0    1
 $EndComp
-$Comp
-L power:+3.3V #PWR010
-U 1 1 5BA42FDB
-P 2550 3350
-F 0 "#PWR010" H 2550 3200 50  0001 C CNN
-F 1 "+3.3V" H 2565 3523 50  0000 C CNN
-F 2 "" H 2550 3350 50  0001 C CNN
-F 3 "" H 2550 3350 50  0001 C CNN
-	1    2550 3350
-	1    0    0    -1
-$EndComp
-Wire Wire Line
-	2550 3350 2550 3450
-Wire Wire Line
-	2650 3850 2650 4050
 Connection ~ 2650 4050
 Wire Wire Line
@@
 F 0 "C3" H 5492 1296 50  0000 L CNN
 F 1 "10uF" H 5492 1205 50  0000 L CNN
-F 2 "Capacitors_SMD:C_0805_HandSoldering" H 5400 1250 50  0001 C CNN
+F 2 "Capacitor_SMD:C_0805_2012Metric" H 5400 1250 50  0001 C CNN
 F 3 "~" H 5400 1250 50  0001 C CNN
 	1    5400 1250
@@
 Wire Wire Line
 	2450 4150 2550 4150
-Wire Wire Line
-	2750 3850 2750 3950
 Connection ~ 2750 3950
 Wire Wire Line
 	2750 3950 2950 3950
-Wire Wire Line
-	2550 3850 2550 4150
 Connection ~ 2550 4150
 Wire Wire Line
 	2550 4150 2950 4150
-Wire Wire Line
-	2550 3450 2650 3450
-Connection ~ 2550 3450
-Wire Wire Line
-	2650 3450 2750 3450
-Connection ~ 2650 3450
-Wire Wire Line
-	2750 3450 2850 3450
-Connection ~ 2750 3450
 Text Label 2300 2550 0    50   ~ 0
 SDA
@@
 F 0 "C4" H 5892 1296 50  0000 L CNN
 F 1 "10uF" H 5892 1205 50  0000 L CNN
-F 2 "Capacitors_SMD:C_0805_HandSoldering" H 5800 1250 50  0001 C CNN
+F 2 "Capacitor_SMD:C_0805_2012Metric" H 5800 1250 50  0001 C CNN
 F 3 "~" H 5800 1250 50  0001 C CNN
 	1    5800 1250
@@
 	5400 1350 5800 1350
 Connection ~ 5400 1350
+Wire Wire Line
+	2550 4300 2550 4150
+Wire Wire Line
+	2650 4050 2650 4300
+Wire Wire Line
+	2750 4300 2750 3950
+$Comp
+L power:GND #PWR0101
+U 1 1 5BC190CF
+P 2750 4700
+F 0 "#PWR0101" H 2750 4450 50  0001 C CNN
+F 1 "GND" H 2755 4527 50  0000 C CNN
+F 2 "" H 2750 4700 50  0001 C CNN
+F 3 "" H 2750 4700 50  0001 C CNN
+	1    2750 4700
+	1    0    0    -1
+$EndComp
+Wire Wire Line
+	2750 4700 2650 4700
+Connection ~ 2750 4700
+Wire Wire Line
+	2650 4700 2550 4700
+Connection ~ 2650 4700
+$Comp
+L Switch:SW_DIP_x06 SW1
+U 1 1 5BC21FF9
+P 2200 1350
+F 0 "SW1" H 2200 1917 50  0000 C CNN
+F 1 "SW_DIP_x06" H 2200 1826 50  0000 C CNN
+F 2 "Buttons_Switches_SMD:SW_DIP_x6_W5.08mm_Slide_Copal_CHS-A" H 2200 1350 50  0001 C CNN
+F 3 "" H 2200 1350 50  0001 C CNN
+	1    2200 1350
+	1    0    0    -1
+$EndComp
+$Comp
+L power:+3.3V #PWR0102
+U 1 1 5BC2887B
+P 1900 1000
+F 0 "#PWR0102" H 1900 850 50  0001 C CNN
+F 1 "+3.3V" H 1915 1173 50  0000 C CNN
+F 2 "" H 1900 1000 50  0001 C CNN
+F 3 "" H 1900 1000 50  0001 C CNN
+	1    1900 1000
+	1    0    0    -1
+$EndComp
+Wire Wire Line
+	2500 1250 2750 1250
+Wire Wire Line
+	2500 1150 2650 1150
+Wire Wire Line
+	2500 1050 2550 1050
+Text Label 3100 1550 0    50   ~ 0
+A0
+Text Label 3100 1450 0    50   ~ 0
+A1
+Text Label 3100 1350 0    50   ~ 0
+A2
+Wire Wire Line
+	1900 1000 1900 1050
+Wire Wire Line
+	1900 1050 1900 1150
+Connection ~ 1900 1050
+Wire Wire Line
+	1900 1150 1900 1250
+Connection ~ 1900 1150
+Wire Wire Line
+	1900 1250 1900 1350
+Connection ~ 1900 1250
+Wire Wire Line
+	1900 1350 1900 1450
+Connection ~ 1900 1350
+Wire Wire Line
+	1900 1450 1900 1550
+Connection ~ 1900 1450
+Wire Wire Line
+	2550 1050 2550 2050
+Wire Wire Line
+	2650 1150 2650 2050
+Wire Wire Line
+	2500 1550 3300 1550
+Wire Wire Line
+	2500 1450 3300 1450
+Wire Wire Line
+	2500 1350 3300 1350
+Wire Wire Line
+	2750 2050 2750 1250
 $EndSCHEMATC

Commit message: - Added a dip switch for setting the address and termination - Added mounting holes - Changed J1 to a 10-pin connector with all pins duplicated   for stacking - Minor cleanup - Updated README
Signed-off-by: Aaron Williams <aaron.w2@gmail.com>
Parts:
- removed J1: Conn_01x06, Pin_Headers:Pin_Header_Angled_1x06_Pitch2.54mm, symbol Connector:Conn_01x06
- added FID1, FID4: FIDUCIAL_1MM, Fiducial:Fiducial_1mm_Dia_2.54mm_Outer_CopperTop, symbol fiducial:FIDUCIAL_1MM
- added FID2, FID3: FIDUCIAL_1MM, Fiducial:Fiducial_1mm_Dia_2.54mm_Outer_CopperBottom, symbol fiducial:FIDUCIAL_1MM
- added J1: Conn_01x10, Pin_Headers:Pin_Header_Angled_1x10_Pitch2.54mm, symbol Connector_Generic:Conn_01x10
- added MH1, MH2: MountingHole, MountingHole:MountingHole_2.5mm, symbol Mechanical:MountingHole
- SW1: footprint Buttons_Switches_SMD:SW_DIP_x6_W5.08mm_Slide_Copal_CHS-A -> Aaron:SW_DIP_SPSTx06_Slide_GrayHill_97C06_W4.5mm_P1.27mm
Connections:
- net labels added: SCL_PU, SDA_PU, ~INT_PU
- wire segments 90 -> 99
Changed lines of the file:
@@
-$EndComp
-$Comp
-L Connector:Conn_01x06 J1
-U 1 1 5BA21BE7
-P 2000 2750
-F 0 "J1" H 1920 2225 50  0000 C CNN
-F 1 "Conn_01x06" H 1920 2316 50  0000 C CNN
-F 2 "Pin_Headers:Pin_Header_Angled_1x06_Pitch2.54mm" H 2000 2750 50  0001 C CNN
-F 3 "~" H 2000 2750 50  0001 C CNN
-	1    2000 2750
-	-1   0    0    1
 $EndComp
 $Comp
@@
 Wire Wire Line
 	2250 2050 2250 2450
-Wire Wire Line
-	2250 2450 2200 2450
 $Comp
 L power:GND #PWR08
 U 1 1 5BA223A1
-P 2200 3150
-F 0 "#PWR08" H 2200 2900 50  0001 C CNN
-F 1 "GND" H 2205 2977 50  0000 C CNN
-F 2 "" H 2200 3150 50  0001 C CNN
-F 3 "" H 2200 3150 50  0001 C CNN
-	1    2200 3150
-	1    0    0    -1
-$EndComp
-Wire Wire Line
-	2200 3150 2200 2950
-Wire Wire Line
-	2200 2950 2200 2850
-Connection ~ 2200 2950
+P 2100 3650
+F 0 "#PWR08" H 2100 3400 50  0001 C CNN
+F 1 "GND" H 2105 3477 50  0000 C CNN
+F 2 "" H 2100 3650 50  0001 C CNN
+F 3 "" H 2100 3650 50  0001 C CNN
+	1    2100 3650
+	1    0    0    -1
+$EndComp
 $Comp
 L Device:C_Small C1
@@
 $EndComp
 Wire Wire Line
-	2450 4050 2650 4050
+	2450 4050 2550 4050
 $Comp
 L Device:R_Pack04 RN2
@@
 	1    0    0    1
 $EndComp
-Connection ~ 2650 4050
-Wire Wire Line
-	2650 4050 2950 4050
 $Comp
 L Device:C_Small C3
@@
 	4950 1350 5400 1350
 Wire Wire Line
-	2200 2750 2550 2750
-Wire Wire Line
 	2750 2450 2750 2650
 Connection ~ 2750 2650
@@
 	2750 2650 2950 2650
 Wire Wire Line
-	2200 2650 2750 2650
-Wire Wire Line
 	2650 2450 2650 2550
 Connection ~ 2650 2550
 Wire Wire Line
-	2200 2550 2650 2550
-Wire Wire Line
 	2550 2450 2550 2750
 Connection ~ 2550 2750
 Wire Wire Line
 	2550 2750 2950 2750
-Wire Wire Line
-	2450 3950 2750 3950
-Wire Wire Line
-	2450 4150 2550 4150
-Connection ~ 2750 3950
-Wire Wire Line
-	2750 3950 2950 3950
-Connection ~ 2550 4150
-Wire Wire Line
-	2550 4150 2950 4150
 Text Label 2300 2550 0    50   ~ 0
 SDA
@@
 	5400 1350 5800 1350
 Connection ~ 5400 1350
-Wire Wire Line
-	2550 4300 2550 4150
-Wire Wire Line
-	2650 4050 2650 4300
-Wire Wire Line
-	2750 4300 2750 3950
 $Comp
 L power:GND #PWR0101
 U 1 1 5BC190CF
-P 2750 4700
-F 0 "#PWR0101" H 2750 4450 50  0001 C CNN
-F 1 "GND" H 2755 4527 50  0000 C CNN
-F 2 "" H 2750 4700 50  0001 C CNN
-F 3 "" H 2750 4700 50  0001 C CNN
-	1    2750 4700
-	1    0    0    -1
-$EndComp
-Wire Wire Line
-	2750 4700 2650 4700
-Connection ~ 2750 4700
+P 2450 4700
+F 0 "#PWR0101" H 2450 4450 50  0001 C CNN
+F 1 "GND" H 2455 4527 50  0000 C CNN
+F 2 "" H 2450 4700 50  0001 C CNN
+F 3 "" H 2450 4700 50  0001 C CNN
+	1    2450 4700
+	1    0    0    -1
+$EndComp
 Wire Wire Line
 	2650 4700 2550 4700
-Connection ~ 2650 4700
 $Comp
 L Switch:SW_DIP_x06 SW1
@@
 F 0 "SW1" H 2200 1917 50  0000 C CNN
 F 1 "SW_DIP_x06" H 2200 1826 50  0000 C CNN
-F 2 "Buttons_Switches_SMD:SW_DIP_x6_W5.08mm_Slide_Copal_CHS-A" H 2200 1350 50  0001 C CNN
+F 2 "Aaron:SW_DIP_SPSTx06_Slide_GrayHill_97C06_W4.5mm_P1.27mm" H 2200 1350 50  0001 C CNN
 F 3 "" H 2200 1350 50  0001 C CNN
 	1    2200 1350
@@
 Wire Wire Line
 	2750 2050 2750 1250
+Wire Wire Line
+	2550 2750 2550 3250
+Wire Wire Line
+	2750 2650 2750 3150
+Text Label 2550 2000 1    50   ~ 0
+~INT_PU
+Text Label 2650 2000 1    50   ~ 0
+SCL_PU
+Text Label 2750 2000 1    50   ~ 0
+SDA_PU
+Wire Wire Line
+	2450 4300 2450 4150
+Wire Wire Line
+	2450 4150 2950 4150
+Wire Wire Line
+	2550 4300 2550 4050
+Connection ~ 2550 4050
+Wire Wire Line
+	2550 4050 2950 4050
+Wire Wire Line
+	2450 3950 2650 3950
+Wire Wire Line
+	2650 4300 2650 3950
+Connection ~ 2650 3950
+Wire Wire Line
+	2650 3950 2950 3950
+Wire Wire Line
+	2450 4700 2550 4700
+Connection ~ 2550 4700
+Connection ~ 2450 4700
+$Comp
+L fiducial:FIDUCIAL_1MM FID1
+U 1 1 5BB5BAAB
+P 7000 1000
+F 0 "FID1" H 7103 1106 60  0000 L CNN
+F 1 "FIDUCIAL_1MM" H 7103 1000 60  0000 L CNN
+F 2 "Fiducial:Fiducial_1mm_Dia_2.54mm_Outer_CopperTop" H 7103 894 60  0000 L CNN
+F 3 "" H 7000 1000 60  0000 C CNN
+	1    7000 1000
+	1    0    0    -1
+$EndComp
+$Comp
+L fiducial:FIDUCIAL_1MM FID2
+U 1 1 5BB5BD3A
+P 7000 1300
+F 0 "FID2" H 7103 1406 60  0000 L CNN
+F 1 "FIDUCIAL_1MM" H 7103 1300 60  0000 L CNN
+F 2 "Fiducial:Fiducial_1mm_Dia_2.54mm_Outer_CopperBottom" H 7103 1194 60  0000 L CNN
+F 3 "" H 7000 1300 60  0000 C CNN
+	1    7000 1300
+	1    0    0    -1
+$EndComp
+$Comp
+L fiducial:FIDUCIAL_1MM FID3
+U 1 1 5BB61DDE
+P 7000 1650
+F 0 "FID3" H 7103 1756 60  0000 L CNN
+F 1 "FIDUCIAL_1MM" H 7103 1650 60  0000 L CNN
+F 2 "Fiducial:Fiducial_1mm_Dia_2.54mm_Outer_CopperBottom" H 7103 1544 60  0000 L CNN
+F 3 "" H 7000 1650 60  0000 C CNN
+	1    7000 1650
+	1    0    0    -1
+$EndComp
+$Comp
+L fiducial:FIDUCIAL_1MM FID4
+U 1 1 5BB61F40
+P 7000 1950
+F 0 "FID4" H 7103 2056 60  0000 L CNN
+F 1 "FIDUCIAL_1MM" H 7103 1950 60  0000 L CNN
+F 2 "Fiducial:Fiducial_1mm_Dia_2.54mm_Outer_CopperTop" H 7103 1844 60  0000 L CNN
+F 3 "" H 7000 1950 60  0000 C CNN
+	1    7000 1950
+	1    0    0    -1
+$EndComp
+$Comp
+L Connector_Generic:Conn_01x10 J1
+U 1 1 5BB62464
+P 1800 2950
+F 0 "J1" H 1720 2225 50  0000 C CNN
+F 1 "Conn_01x10" H 1720 2316 50  0000 C CNN
+F 2 "Pin_Headers:Pin_Header_Angled_1x10_Pitch2.54mm" H 1800 2950 50  0001 C CNN
+F 3 "~" H 1800 2950 50  0001 C CNN
+	1    1800 2950
+	-1   0    0    1
+$EndComp
+Wire Wire Line
+	2000 2450 2250 2450
+Wire Wire Line
+	2000 2550 2650 2550
+Wire Wire Line
+	2000 2650 2750 2650
+Wire Wire Line
+	2000 2750 2550 2750
+Wire Wire Line
+	2100 3650 2100 3350
+Wire Wire Line
+	2100 2850 2000 2850
+Wire Wire Line
+	2000 2950 2250 2950
+Wire Wire Line
+	2250 2950 2250 2450
+Connection ~ 2250 2450
+Wire Wire Line
+	2000 3050 2650 3050
+Wire Wire Line
+	2650 3050 2650 2550
+Wire Wire Line
+	2750 3150 2000 3150
+Wire Wire Line
+	2000 3250 2550 3250
+Wire Wire Line
+	2000 3350 2100 3350
+Connection ~ 2100 3350
+Wire Wire Line
+	2100 3350 2100 2850
+$Comp
+L Mechanical:MountingHole MH2
+U 1 1 5BB8C115
+P 7000 2550
+F 0 "MH2" H 7100 2596 50  0000 L CNN
+F 1 "MountingHole" H 7100 2505 50  0000 L CNN
+F 2 "MountingHole:MountingHole_2.5mm" H 7000 2550 50  0001 C CNN
+F 3 "~" H 7000 2550 50  0001 C CNN
+	1    7000 2550
+	1    0    0    -1
+$EndComp
+$Comp
+L Mechanical:MountingHole MH1
+U 1 1 5BB8F6EA
+P 7000 2300
+F 0 "MH1" H 7100 2346 50  0000 L CNN
+F 1 "MountingHole" H 7100 2255 50  0000 L CNN
+F 2 "MountingHole:MountingHole_2.5mm" H 7000 2300 50  0001 C CNN
+F 3 "~" H 7000 2300 50  0001 C CNN
+	1    7000 2300
+	1    0    0    -1
+$EndComp
 $EndSCHEMATC

Commit message: Fixed solder mask clearance.
Signed-off-by: Aaron Williams <aaron.w2@gmail.com>
Parts:
- removed RN1: 10k, Resistor_SMD:R_Array_Convex_4x0603, symbol Device:R_Pack04
- added RN1: R_Pack02, Resistor_SMD:R_Array_Concave_2x0603, symbol device:R_Pack02
- U1: footprint Housings_SSOP:SOIC-24_5.3x6.2mm_Pitch0.65 -> Housings_SSOP:TSSOP-24_4.4x7.8mm_Pitch0.65mm
Connections:
- wire segments 99 -> 98
Changed lines of the file:
@@
 F 0 "U1" H 3300 4300 50  0000 C CNN
 F 1 "TCA9555DBT" H 3900 4300 50  0000 C CNN
-F 2 "Housings_SSOP:SOIC-24_5.3x6.2mm_Pitch0.65" H 4700 2350 50  0001 C CNN
+F 2 "Housings_SSOP:TSSOP-24_4.4x7.8mm_Pitch0.65mm" H 4700 2350 50  0001 C CNN
 F 3 "http://www.ti.com/lit/ds/symlink/tca9555.pdf" H 3150 4250 50  0001 C CNN
 	1    3650 3350
@@
 	1    0    0    -1
 $EndComp
-Wire Wire Line
-	2950 2550 2650 2550
 Wire Wire Line
 	2250 2050 2250 2450
@@
 P17
 $Comp
-L Device:R_Pack04 RN1
-U 1 1 5BA38513
-P 2750 2250
-F 0 "RN1" H 2938 2296 50  0000 L CNN
-F 1 "10k" H 2938 2205 50  0000 L CNN
-F 2 "Resistor_SMD:R_Array_Convex_4x0603" V 3025 2250 50  0001 C CNN
-F 3 "~" H 2750 2250 50  0001 C CNN
-	1    2750 2250
-	1    0    0    -1
-$EndComp
-Wire Wire Line
-	2450 4050 2550 4050
-$Comp
 L Device:R_Pack04 RN2
 U 1 1 5BA42F5D
@@
 Wire Wire Line
 	4950 1350 5400 1350
-Wire Wire Line
-	2750 2450 2750 2650
-Connection ~ 2750 2650
-Wire Wire Line
-	2750 2650 2950 2650
-Wire Wire Line
-	2650 2450 2650 2550
-Connection ~ 2650 2550
-Wire Wire Line
-	2550 2450 2550 2750
 Connection ~ 2550 2750
 Wire Wire Line
@@
 	1    0    0    -1
 $EndComp
-Wire Wire Line
-	2650 4700 2550 4700
 $Comp
 L Switch:SW_DIP_x06 SW1
@@
 $EndComp
 Wire Wire Line
-	2500 1250 2750 1250
-Wire Wire Line
 	2500 1150 2650 1150
 Wire Wire Line
 	2500 1050 2550 1050
-Text Label 3100 1550 0    50   ~ 0
-A0
 Text Label 3100 1450 0    50   ~ 0
 A1
-Text Label 3100 1350 0    50   ~ 0
-A2
 Wire Wire Line
 	1900 1000 1900 1050
@@
 	2500 1350 3300 1350
 Wire Wire Line
-	2750 2050 2750 1250
-Wire Wire Line
 	2550 2750 2550 3250
-Wire Wire Line
-	2750 2650 2750 3150
 Text Label 2550 2000 1    50   ~ 0
 ~INT_PU
 Text Label 2650 2000 1    50   ~ 0
-SCL_PU
-Text Label 2750 2000 1    50   ~ 0
 SDA_PU
 Wire Wire Line
-	2450 4300 2450 4150
-Wire Wire Line
-	2450 4150 2950 4150
-Wire Wire Line
 	2550 4300 2550 4050
-Connection ~ 2550 4050
 Wire Wire Line
 	2550 4050 2950 4050
-Wire Wire Line
-	2450 3950 2650 3950
-Wire Wire Line
-	2650 4300 2650 3950
-Connection ~ 2650 3950
-Wire Wire Line
-	2650 3950 2950 3950
-Wire Wire Line
-	2450 4700 2550 4700
-Connection ~ 2550 4700
-Connection ~ 2450 4700
 $Comp
 L fiducial:FIDUCIAL_1MM FID1
@@
 	2000 2450 2250 2450
 Wire Wire Line
-	2000 2550 2650 2550
-Wire Wire Line
-	2000 2650 2750 2650
-Wire Wire Line
 	2000 2750 2550 2750
 Wire Wire Line
@@
 	2250 2950 2250 2450
 Connection ~ 2250 2450
-Wire Wire Line
-	2000 3050 2650 3050
-Wire Wire Line
-	2650 3050 2650 2550
-Wire Wire Line
-	2750 3150 2000 3150
 Wire Wire Line
 	2000 3250 2550 3250
@@
 	1    0    0    -1
 $EndComp
+Text Label 3100 1350 0    50   ~ 0
+A0
+Text Label 3100 1550 0    50   ~ 0
+A2
+Wire Wire Line
+	2450 3950 2950 3950
+Wire Wire Line
+	2450 3950 2450 4300
+Wire Wire Line
+	2950 4150 2650 4150
+Wire Wire Line
+	2650 4150 2650 4300
+Wire Wire Line
+	2750 4700 2750 5000
+Wire Wire Line
+	2750 5000 3150 5000
+Text Label 2750 4300 0    50   ~ 0
+SCL_PU
+Wire Wire Line
+	2500 1250 3300 1250
+Text Label 3000 1250 0    50   ~ 0
+SCL_PU
+Wire Wire Line
+	2750 4300 3050 4300
+Text Label 2900 5000 0    50   ~ 0
+SCL
+$Comp
+L device:R_Pack02 RN1
+U 1 1 5BBC208F
+P 2650 2250
+F 0 "RN1" H 2738 2296 50  0000 L CNN
+F 1 "R_Pack02" H 2738 2205 50  0000 L CNN
+F 2 "Resistor_SMD:R_Array_Concave_2x0603" V 2825 2250 50  0001 C CNN
+F 3 "" H 2650 2250 50  0001 C CNN
+	1    2650 2250
+	1    0    0    -1
+$EndComp
+Wire Wire Line
+	2550 2450 2550 2750
+Wire Wire Line
+	2000 2550 2650 2550
+Wire Wire Line
+	2000 3050 2650 3050
+Wire Wire Line
+	2650 2450 2650 2550
+Connection ~ 2650 2550
+Wire Wire Line
+	2650 4700 2550 4700
+Wire Wire Line
+	2550 4700 2450 4700
+Connection ~ 2550 4700
+Connection ~ 2450 4700
+Wire Wire Line
+	2650 2550 2650 3050
+Wire Wire Line
+	2650 2550 2950 2550
+Wire Wire Line
+	2750 3150 2750 2650
+Connection ~ 2750 2650
+Wire Wire Line
+	2750 2650 2950 2650
+Wire Wire Line
+	2000 3150 2750 3150
+Wire Wire Line
+	2000 2650 2750 2650
 $EndSCHEMATC

Commit message: Fixed the footprint to not use a git library.
Signed-off-by: Aaron Williams <aaron.w2@gmail.com>
Parts:
- U1: footprint Housings_SSOP:TSSOP-24_4.4x7.8mm_Pitch0.65mm -> Package_SO:TSSOP-24_4.4x7.8mm_P0.65mm
Changed lines of the file:
@@
 F 0 "U1" H 3300 4300 50  0000 C CNN
 F 1 "TCA9555DBT" H 3900 4300 50  0000 C CNN
-F 2 "Housings_SSOP:TSSOP-24_4.4x7.8mm_Pitch0.65mm" H 4700 2350 50  0001 C CNN
+F 2 "Package_SO:TSSOP-24_4.4x7.8mm_P0.65mm" H 4700 2350 50  0001 C CNN
 F 3 "http://www.ti.com/lit/ds/symlink/tca9555.pdf" H 3150 4250 50  0001 C CNN
 	1    3650 3350
